Commit message: Added depthimage_to_laserscan converter node into launchfile

File: grvc-ual/robots_description/models/mbzirc/geometry.xacro (robot description, xacro)
@@ -211,3 +211,40 @@
     <xacro:insert_block name="rotor_inertia" />
   </xacro:vertical_rotor>
+  <!-- <include filename="$(find velodyne_description)/urdf/VLP-16.urdf.xacro" /> -->
+  <!-- <xacro:VLP-16 robot_namespace="${namespace}"
+    name="laser_scan"
+    parent="base"
+    ros_topic="base_scan/scan"
+    update_rate="20"
+    min_angle="-1.57"
+    max_angle="1.57" >
+    <origin xyz="${0.4 - 0.01 - 0.04} 0 0.3" rpy="0 0 0" />
+  </xacro:VLP-16> -->
+      <!-- This adds a visual box to allow us to see the Hokuyo in rviz/gazebo -->
+      <!-- <joint name="laser_joint" type="fixed">
+          <origin xyz="0.0 0 0.05" rpy="0 0 0" />
+          <parent link="base_link" />
+          <child link="laser_link"/>
+      </joint>
+      <link name="laser_link">
+          <inertial>
+              <mass value="0.01" />
+              <origin xyz="0 0 0" />
+              <inertia ixx="0.001"  ixy="0.0"  ixz="0.0"
+              iyy="0.001"  iyz="0.0"
+                  izz="0.001" />
+              </inertial>
+              <visual>
+                  <origin xyz="0 0 0" rpy="0 0 0"/>
+                  <geometry>
+                      <box size="0.05 0.05 0.1" />
+                  </geometry>
+              </visual>
+              <collision>
+                  <origin xyz="0 0 0" rpy="0 0 0"/>
+                  <geometry>
+                      <box size="0.05 0.05 0.1" />
+                  </geometry>
+              </collision>
+          </link> -->
 </robot>
