Commit message: [sim] Adjusting sensor height, laser number and view angle.

File: architecture/Tools/iris.xacro (robot description, xacro)
@@ -138,6 +138,6 @@
   </xacro:vertical_rotor>
   <xacro:include filename="/opt/ros/kinetic/share/velodyne_description/urdf/VLP-16.urdf.xacro"/>
-  <VLP-16 parent="base_link" name="velodyne" topic="/velodyne_points" hz="10" samples="440" lasers="5" max_range="10">
-    <origin xyz="0 0 1" rpy="0 0 0" />
+  <VLP-16 parent="base_link" name="velodyne" topic="/velodyne_points" hz="10" samples="440" lasers="2" min_angle="-2.35619" max_angle="2.35619" max_range="10">
+    <origin xyz="0 0 0.04" rpy="0 0 0" />
   </VLP-16>
 </robot>

File: architecture/Tools/iris_base.urdf (robot description, URDF)
Before this commit: robot iris, 9 links, 8 joints
Joints:
- joint velodyne_base_mount_joint: origin xyz=0 0 1 rpy=0 0 0 -> xyz=0 0 0.04 rpy=0 0 0

File: architecture/Tools/iris_base.xacro (robot description, xacro)
@@ -128,3 +128,15 @@
     </gazebo>
   </xacro:if>
+  <gazebo>
+      <plugin name="ground_truth" filename="libgazebo_ros_p3d.so">
+        <alwaysOn>true</alwaysOn>
+        <frameName>map</frameName>
+        <topicName>ground_truth_pose</topicName>
+        <bodyName>base_link</bodyName>
+        <updateRate>100.0</updateRate>
+        <xyzOffsets>5 5 0</xyzOffsets> <!-- initialize odometry for fake localization-->
+        <rpyOffsets>0 0 0</rpyOffsets>
+<!--        <interface:position name="p3d_base_position"/>  -->
+      </plugin>
+    </gazebo>
 </robot>

Commit message: [architecture] Tilt the sensor so it can explore more in z.

File: architecture/Tools/iris.xacro (robot description, xacro)
@@ -140,5 +140,5 @@
   <!-- <VLP-16 parent="base_link" name="velodyne" topic="/velodyne_points" hz="10" samples="440" lasers="16" min_angle="-2.35619" max_angle="2.35619" max_range="10"> -->
   <VLP-16 parent="base_link" name="velodyne" topic="/velodyne_points" hz="10" samples="440" lasers="16" min_angle="-3.14" max_angle="3.14" max_range="10">
-    <origin xyz="0 0 0.04" rpy="0 0 0" />
+    <origin xyz="0 0 0.05" rpy="0 0.174533 0" />
   </VLP-16>
 </robot>

Commit message: [architecture] Adding sensor model.

File: architecture/Tools/iris.xacro (robot description, xacro)
@@ -137,8 +137,69 @@
     <xacro:insert_block name="rotor_inertia" />
   </xacro:vertical_rotor>
-  <xacro:include filename="/opt/ros/kinetic/share/velodyne_description/urdf/VLP-16.urdf.xacro"/>
-  <!-- <VLP-16 parent="base_link" name="velodyne" topic="/velodyne_points" hz="10" samples="440" lasers="16" min_angle="-2.35619" max_angle="2.35619" max_range="10"> -->
+  <!-- <xacro:include filename="/opt/ros/kinetic/share/velodyne_description/urdf/VLP-16.urdf.xacro"/>
+  <VLP-16 parent="base_link" name="velodyne" topic="/velodyne_points" hz="10" samples="440" lasers="16" min_angle="-2.35619" max_angle="2.35619" max_range="10">
   <VLP-16 parent="base_link" name="velodyne" topic="/velodyne_points" hz="10" samples="440" lasers="16" min_angle="-3.14" max_angle="3.14" max_range="10">
     <origin xyz="0 0 0.05" rpy="0 0.174533 0" />
-  </VLP-16>
+  </VLP-16> -->
+  <joint name="hokuyo_joint" type="fixed">
+    <axis xyz="0 1 0" />
+    <origin xyz=".15 0 .1" rpy="0 0 0"/>
+    <parent link="base_link"/>
+    <child link="hokuyo"/>
+  </joint>
+  <!-- Hokuyo Laser -->
+  <link name="hokuyo">
+    <collision>
+      <origin xyz="0 0 0.05" rpy="0 0.174533 0" />
+      <geometry>
+    <box size="0.1 0.1 0.1"/>
+      </geometry>
+    </collision>
+    <visual>
+      <origin xyz="0 0 0.05" rpy="0 0.174533 0" />
+      <geometry>
+        <mesh filename="package://architecture/meshes/hokuyo.dae"/>
+      </geometry>
+    </visual>
+    <inertial>
+      <mass value="1e-5" />
+      <origin xyz="0 0 0" rpy="0 0 0"/>
+      <inertia ixx="1e-6" ixy="0" ixz="0" iyy="1e-6" iyz="0" izz="1e-6" />
+    </inertial>
+  </link>
+  <gazebo reference="hokuyo">
+    <sensor type="ray" name="head_hokuyo_sensor">
+      <pose>0 0 0 0 0 0</pose>
+      <visualize>true</visualize>
+      <update_rate>40</update_rate>
+      <ray>
+        <scan>
+          <horizontal>
+            <samples>720</samples>
+            <resolution>1</resolution>
+            <min_angle>-1.570796</min_angle>
+            <max_angle>1.570796</max_angle>
+          </horizontal>
+        </scan>
+        <range>
+          <min>0.10</min>
+          <max>30.0</max>
+          <resolution>0.01</resolution>
+        </range>
+        <noise>
+          <type>gaussian</type>
+          <!-- Noise parameters based on published spec for Hokuyo laser
+               achieving "+-30mm" accuracy at range < 10m.  A mean of 0.0m and
+               stddev of 0.01m will put 99.7% of samples within 0.03m of the true
+               reading. -->
+          <mean>0.0</mean>
+          <stddev>0.01</stddev>
+        </noise>
+      </ray>
+      <plugin name="gazebo_ros_head_hokuyo_controller" filename="libgazebo_ros_laser.so">
+        <topicName>/mybot/laser/scan</topicName>
+        <frameName>hokuyo</frameName>
+      </plugin>
+    </sensor>
+  </gazebo>
 </robot>

Commit message: [architecture] Moving the sensor to be more tilted and centered.

File: architecture/Tools/iris.xacro (robot description, xacro)
@@ -144,5 +144,5 @@
   <joint name="hokuyo_joint" type="fixed">
     <axis xyz="0 1 0" />
-    <origin xyz=".15 0 .1" rpy="0 0 0"/>
+    <origin xyz="0 0 .1" rpy="0 -0.261799 3.14"/>
     <parent link="base_link"/>
     <child link="hokuyo"/>
@@ -151,5 +151,5 @@
   <link name="hokuyo">
     <collision>
-      <origin xyz="0 0 0.05" rpy="0 0.174533 0" />
+      <origin xyz="0 0 0" rpy="0 0 0" />
       <geometry>
     <box size="0.1 0.1 0.1"/>
@@ -157,5 +157,5 @@
     </collision>
     <visual>
-      <origin xyz="0 0 0.05" rpy="0 0.174533 0" />
+      <origin xyz="0 0 0" rpy="0 0 0" />
       <geometry>
         <mesh filename="package://architecture/meshes/hokuyo.dae"/>

Commit message: [architecture] Checking free voxels for velodyne sensor.

File: architecture/Tools/iris.xacro (robot description, xacro)
@@ -137,17 +137,17 @@
     <xacro:insert_block name="rotor_inertia" />
   </xacro:vertical_rotor>
-  <!-- <xacro:include filename="/opt/ros/kinetic/share/velodyne_description/urdf/VLP-16.urdf.xacro"/>
-  <VLP-16 parent="base_link" name="velodyne" topic="/velodyne_points" hz="10" samples="440" lasers="16" min_angle="-2.35619" max_angle="2.35619" max_range="10">
-  <VLP-16 parent="base_link" name="velodyne" topic="/velodyne_points" hz="10" samples="440" lasers="16" min_angle="-3.14" max_angle="3.14" max_range="10">
+  <xacro:include filename="/opt/ros/kinetic/share/velodyne_description/urdf/VLP-16.urdf.xacro"/>
+  <!-- <VLP-16 parent="base_link" name="velodyne" topic="/velodyne_points" hz="10" samples="440" lasers="16" min_angle="-2.35619" max_angle="2.35619" max_range="10"> -->
+  <VLP-16 parent="base_link" name="velodyne" topic="/velodyne_points" hz="10" samples="440" lasers="16" min_angle="-3.14" max_angle="3.14" max_range="100">
     <origin xyz="0 0 0.05" rpy="0 0.174533 0" />
-  </VLP-16> -->
-  <joint name="hokuyo_joint" type="fixed">
+  </VLP-16>
+  <!-- <joint name="hokuyo_joint" type="fixed">
     <axis xyz="0 1 0" />
     <origin xyz="0 0 .1" rpy="0 -0.261799 3.14"/>
     <parent link="base_link"/>
     <child link="hokuyo"/>
-  </joint>
+  </joint>  -->
   <!-- Hokuyo Laser -->
-  <link name="hokuyo">
+  <!-- <link name="hokuyo">
     <collision>
       <origin xyz="0 0 0" rpy="0 0 0" />
@@ -188,10 +188,10 @@
         </range>
         <noise>
-          <type>gaussian</type>
+          <type>gaussian</type>  -->
           <!-- Noise parameters based on published spec for Hokuyo laser
                achieving "+-30mm" accuracy at range < 10m.  A mean of 0.0m and
                stddev of 0.01m will put 99.7% of samples within 0.03m of the true
                reading. -->
-          <mean>0.0</mean>
+          <!-- <mean>0.0</mean>
           <stddev>0.01</stddev>
         </noise>
@@ -202,4 +202,4 @@
       </plugin>
     </sensor>
-  </gazebo>
+  </gazebo>  -->
 </robot>

Commit message: [gazebo] Switching back to Hokuyo.

File: architecture/Tools/iris.xacro (robot description, xacro)
@@ -137,17 +137,17 @@
     <xacro:insert_block name="rotor_inertia" />
   </xacro:vertical_rotor>
-  <xacro:include filename="/opt/ros/kinetic/share/velodyne_description/urdf/VLP-16.urdf.xacro"/>
+  <!-- <xacro:include filename="/opt/ros/kinetic/share/velodyne_description/urdf/VLP-16.urdf.xacro"/> -->
   <!-- <VLP-16 parent="base_link" name="velodyne" topic="/velodyne_points" hz="10" samples="440" lasers="16" min_angle="-2.35619" max_angle="2.35619" max_range="10"> -->
-  <VLP-16 parent="base_link" name="velodyne" topic="/velodyne_points" hz="10" samples="440" lasers="16" min_angle="-3.14" max_angle="3.14" max_range="100">
+  <!-- <VLP-16 parent="base_link" name="velodyne" topic="/velodyne_points" hz="10" samples="440" lasers="16" min_angle="-3.14" max_angle="3.14" max_range="100">
     <origin xyz="0 0 0.05" rpy="0 0.174533 0" />
-  </VLP-16>
-  <!-- <joint name="hokuyo_joint" type="fixed">
+  </VLP-16> -->
+  <joint name="hokuyo_joint" type="fixed">
     <axis xyz="0 1 0" />
     <origin xyz="0 0 .1" rpy="0 -0.261799 3.14"/>
     <parent link="base_link"/>
     <child link="hokuyo"/>
-  </joint>  -->
+  </joint>
   <!-- Hokuyo Laser -->
-  <!-- <link name="hokuyo">
+  <link name="hokuyo">
     <collision>
       <origin xyz="0 0 0" rpy="0 0 0" />
@@ -188,10 +188,10 @@
         </range>
         <noise>
-          <type>gaussian</type>  -->
+          <type>gaussian</type>
           <!-- Noise parameters based on published spec for Hokuyo laser
                achieving "+-30mm" accuracy at range < 10m.  A mean of 0.0m and
                stddev of 0.01m will put 99.7% of samples within 0.03m of the true
                reading. -->
-          <!-- <mean>0.0</mean>
+          <mean>0.0</mean>
           <stddev>0.01</stddev>
         </noise>
@@ -202,4 +202,4 @@
       </plugin>
     </sensor>
-  </gazebo>  -->
+  </gazebo>
 </robot>

Commit message: [px4] 20 degree tilt.

File: architecture/Tools/iris.xacro (robot description, xacro)
@@ -144,5 +144,5 @@
   <joint name="hokuyo_joint" type="fixed">
     <axis xyz="0 1 0" />
-    <origin xyz="0 0 .1" rpy="0 -0.261799 3.14"/>
+    <origin xyz="0 0 .1" rpy="0 -0.349066 3.14"/>
     <parent link="base_link"/>
     <child link="hokuyo"/>

Commit message: [architecture] [frontier] Now the xy distance to what is whithin reach is calculated according to sensor angle and range. The frontier generation checks if the frontier can be sensed from the center of the frontier voxel, if this is not the case the generated frontier is adjusted to the sensing range. The end goal is added to the pass, instead of going just until the center of containing voxel.

File: architecture/Tools/iris.xacro (robot description, xacro)
@@ -144,5 +144,5 @@
   <joint name="hokuyo_joint" type="fixed">
     <axis xyz="0 1 0" />
-    <origin xyz="0 0 .1" rpy="0 -0.349066 3.14"/>
+    <origin xyz="0 0 .1" rpy="0 -0.872665 3.14"/>
     <parent link="base_link"/>
     <child link="hokuyo"/>
